File: hardware/garageDoor-pro.kicad_pcb (KiCad board)
At the start: 4 copper layers, 60 x 31 mm, 46 parts, among them J1 USB-C, J2 U.FL GNSS antenna, J3 Remote button, K1 CPC1017N, SW1 SETUP, U1 ESP32-C3-MINI-1-H4X, U2 MAX-M10S, U3 AP2112K-3.3, U4 USBLC6-2SC6

Commit message: Hardware: routed, DRC-clean board and JLCPCB order package
- GND/3V3 fanout into solid inner planes, hand-routed 50 ohm GNSS RF path
  and USB VBUS, Freerouting for the remaining signals (inner layers kept as
  planes), outer GND pours and stitching vias
- DRC: 0 violations, 0 unconnected, 0 schematic-parity issues; ERC clean
- production/: Gerbers + Excellon (zip), JLCPCB BOM and CPL, schematic and
  assembly PDFs, 3D renders, STEP
- build.sh regenerates everything from gen/netlist.py

Co-Authored-By: Claude Opus 5.5 <noreply@anthropic.com>
Parts:
- moved TP8 50.9 mm to (108.0, 105.6)
- moved TP9 50.9 mm to (108.0, 107.6)
- moved TP7 42.4 mm to (111.6, 126.4)
- moved TP5 35.2 mm to (118.8, 119.6)
- moved TP6 35.2 mm to (118.8, 121.6)
- moved R6 0.95 mm to (125.2, 111.4)
Routing:
- net /VIN_5V: track 0.00 -> 59.2 mm, vias 0 -> 1
- net GND: track 0.00 -> 45.2 mm, vias 8 -> 136
- net /SWITCH: track 0.00 -> 36.7 mm
- net /BTN_IO9: track 0.00 -> 35.5 mm, vias 0 -> 2
- net /GPS_RESET_N: track 0.00 -> 28.6 mm, vias 0 -> 4
- net /GPS_TX: track 0.00 -> 26.6 mm, vias 0 -> 2
- net /GPS_RX: track 0.00 -> 25.3 mm, vias 0 -> 2
- net /USB_DM: track 0.00 -> 23.2 mm, vias 0 -> 3
- net /GPS_SAFEBOOT: track 0.00 -> 20.4 mm, vias 0 -> 1
- net /USB_DP: track 0.00 -> 20.3 mm
- net /IO2: track 0.00 -> 17.4 mm, vias 0 -> 2
- net /GPS_PPS: track 0.00 -> 17.1 mm, vias 0 -> 1
- net /VBUS: track 0.00 -> 15.9 mm, vias 0 -> 2
- net /LED_STATUS: track 0.00 -> 14.5 mm, vias 0 -> 2
- net +3V3: track 0.00 -> 11.1 mm, vias 0 -> 14
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- added copper zone on B.Cu, net GND
- added copper zone on F.Cu, net GND

Commit message: Firmware, docs and final hardware package
firmware/ (ESP-IDF v6.1, ESP32-C3):
- MAX-M10S over UBX (NAV-PVT 1 Hz, 115200, automotive), reconfigure/reset
  watchdog; trip state machine with home/away memory, arrive/leave
  hysteresis and drive-by detection; PhotoMOS presser; LED codes; SETUP
  button (3 s setup Wi-Fi, 10 s factory reset)
- WPA2 setup AP with captive portal and web panel (set home from GPS or
  coordinates, settings, test press, password, OTA with rollback); the
  panel is locked until the default password is changed
- host unit tests (UBX, geo, trip) under ASan/UBSan; mock panel server
- builds with -Wall -Wextra -Werror, 56 % of the OTA slot free

docs: design.md updated to the as-built design, user guide, JLCPCB
ordering guide with placement checks and a bring-up checklist.

hardware: regenerated from scratch with build.sh, ERC/DRC clean.

Co-Authored-By: Claude Opus 5.5 <noreply@anthropic.com>
Routing:
- net /BTN_IO9: track 35.5 -> 22.6 mm
- net /SWITCH: track 36.7 -> 43.3 mm, vias 0 -> 3
- net /GPS_SAFEBOOT: track 20.4 -> 25.0 mm
- net /CC1: track 9.73 -> 5.54 mm, vias 2 -> 0
- net /VIN_5V: track 59.2 -> 56.2 mm
- net /IO2: track 17.4 -> 19.7 mm, vias 2 -> 4
- net /USB_DP: track 20.3 -> 22.4 mm
- net /GPS_PPS: track 17.1 -> 18.5 mm
- net /GPS_RESET_N: track 28.6 -> 27.3 mm, vias 4 -> 2
- net /LED_STATUS: track 14.5 -> 15.5 mm
- net /USB_DM: track 23.2 -> 22.4 mm
- net /GPS_TX: track 26.6 -> 25.8 mm
- net /GPS_RX: track 25.3 -> 24.7 mm
- net /IO8: track 6.37 -> 6.50 mm, vias 2 -> 0
- net GND: vias 136 -> 131

Commit message: NPN transistor switch everywhere; PCB v1.1 regenerated
The perfboard proved it: the remote's button switches the whole remote
on, and only a transistor driven from GPIO7 carries that current.

- Prototype: Q1 NPN (TO-92: 2N2222, S8050, BC547, ...) in B12/C12/D12,
  straight trails for base, GND/emitter and collector, new pictures,
  leg-order table, measurements and bench test for the transistor.
- PCB: SS8050 (SOT-23, LCSC C2150) replaces the CPC1017N; J3 pin 2 is
  GND, silkscreen marks + / - and says v1.1. Schematic, PCB, routing,
  Gerbers, BOM, CPL, PDFs, renders and STEP regenerated; ERC and DRC clean.
  route.py drops router vias left with copper on one layer only.
- Docs and firmware comments: transistor and polarity (+ to screw 1)
  everywhere; no references to local folders.

Co-Authored-By: Claude Opus 5.5 <noreply@anthropic.com>
Parts:
- removed K1: CPC1017N, Package_SO:SOP-4_3.8x4.1mm_P2.54mm
- added Q1: SS8050, Package_TO_SOT_SMD:SOT-23, F.Cu at (128.5, 126.0)
Connections:
- J3 pad 1: /OUT_A -> /REMOTE_PLUS
- J3 pad 2: /OUT_B -> GND
- R8 pad 2: /K1_LED_A -> /Q1_BASE
Routing:
- net /OUT_B: track 11.0 -> 0.00 mm
- net /Q1_BASE: track 0.00 -> 7.79 mm, vias 0 -> 2
- net /SWITCH: track 43.3 -> 36.2 mm, vias 3 -> 2
- net /REMOTE_PLUS: track 0.00 -> 6.81 mm
- net /BTN_IO9: track 22.6 -> 28.0 mm, vias 2 -> 3
- net /USB_DM: track 22.4 -> 27.7 mm
- net /OUT_A: track 5.03 -> 0.00 mm
- net /GPS_SAFEBOOT: track 25.0 -> 20.4 mm
- net /VIN_5V: track 56.2 -> 60.6 mm
- net /K1_LED_A: track 4.30 -> 0.00 mm
- net /IO2: track 19.7 -> 16.2 mm, vias 4 -> 2
- net /GPS_TX: track 25.8 -> 27.6 mm, vias 2 -> 4
- net /LED_STATUS: track 15.5 -> 13.9 mm
- net /GPS_PPS: track 18.5 -> 17.1 mm
- net /CC1: track 5.54 -> 4.20 mm
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Other:
- board text added: "+"
- board text added: "-"
- board text added: "garageDoor-pro v1.1"
- board text removed: "garageDoor-pro v1.0"
