File: hardware/garageDoor-pro.kicad_sch (KiCad schematic)
At the start: 46 parts, among them J1 USB-C, J2 U.FL GNSS antenna, J3 Remote button, K1 CPC1017N, SW1 SETUP, U1 ESP32-C3-MINI-1-H4X, U2 MAX-M10S, U3 AP2112K-3.3, U4 USBLC6-2SC6

Commit message: NPN transistor switch everywhere; PCB v1.1 regenerated
The perfboard proved it: the remote's button switches the whole remote
on, and only a transistor driven from GPIO7 carries that current.

- Prototype: Q1 NPN (TO-92: 2N2222, S8050, BC547, ...) in B12/C12/D12,
  straight trails for base, GND/emitter and collector, new pictures,
  leg-order table, measurements and bench test for the transistor.
- PCB: SS8050 (SOT-23, LCSC C2150) replaces the CPC1017N; J3 pin 2 is
  GND, silkscreen marks + / - and says v1.1. Schematic, PCB, routing,
  Gerbers, BOM, CPL, PDFs, renders and STEP regenerated; ERC and DRC clean.
  route.py drops router vias left with copper on one layer only.
- Docs and firmware comments: transistor and polarity (+ to screw 1)
  everywhere; no references to local folders.

Co-Authored-By: Claude Opus 5.5 <noreply@anthropic.com>
Parts:
- removed K1: CPC1017N, Package_SO:SOP-4_3.8x4.1mm_P2.54mm, symbol Relay_SolidState:CPC1017N
- added Q1: SS8050, Package_TO_SOT_SMD:SOT-23, symbol Transistor_BJT:SS8050
Connections:
- net OUT_B is gone; now on net GND: J3.2 (Pin_2)
- net GND: now also Q1.2 (E)
- net K1_LED_A renamed Q1_BASE
- net Q1_BASE: now also Q1.1 (B)
- net OUT_A renamed REMOTE_PLUS
- net REMOTE_PLUS: now also Q1.3 (C)
Other:
- note added: "Switch output: SS8050 NPN transistor -> screw terminal to the remote's button (+ to pin 1, - to pin 2)"
- note removed: "Switch output: CPC1017N PhotoMOS -> screw terminal to the remote's button (either polarity)"
